File: Pawn.brd (EAGLE design)
At the start: 90 x 43 mm, 52 parts, among them CON2 MTDRV-A, CON26 MINI-USB-, CON27 UART-S, CON4 D-3500-4, CON5 MOLEX-5251-03-A, CON6 MOLEX-5251-03-A, CON7 MOLEX-5251-02-S_LONG, IC1 AZ1086H-3.3, IC2 7W14FU, IC8 R5F10JB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

Commit message: minor change
Parts:
- C11, C2: value (none) -> 1n
- C17: value (none) -> 0.1u
- R2, R3, R8, R9: value (none) -> 10k
- R4, R5: value (none) -> 1k
Changed lines of the file:
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@@
 <?xml version="1.0" encoding="utf-8"?>
 <!DOCTYPE eagle SYSTEM "eagle.dtd">
-<eagle version="8.5.1">
+<eagle version="8.3.1">
 <drawing>
 <settings>
@@
 <param name="dpMaxLengthDifference" value="10mm"/>
 <param name="dpGapFactor" value="2.5"/>
+<param name="checkGrid" value="0"/>
 <param name="checkAngle" value="1"/>
 <param name="checkFont" value="1"/>
 <param name="checkRestrict" value="1"/>
-<param name="checkStop" value="0"/>
-<param name="checkValues" value="0"/>
 <param name="useDiameter" value="13"/>
 <param name="maxErrors" value="50"/>
@@
 <element name="CON2" library="Connector_Robotech" package="5251-05-A" value="MTDRV-A" x="77" y="21" rot="R270"/>
 <element name="CON4" library="Connector_Robotech" package="D3500D-4-HORIZONTAL" value="D-3500-4" x="4" y="14"/>
-<element name="R2" library="Passive_Robotech" package="2012-R" value="" x="-2" y="11" rot="MR180"/>
-<element name="R3" library="Passive_Robotech" package="2012-R" value="" x="11" y="15" rot="MR90"/>
-<element name="R4" library="Passive_Robotech" package="2012-R" value="" x="10" y="9" rot="MR180"/>
-<element name="R5" library="Passive_Robotech" package="2012-R" value="" x="15" y="15" rot="MR180"/>
-<element name="C2" library="Passive_Robotech" package="2012-C" value="" x="14" y="11" rot="MR270"/>
-<element name="C11" library="Passive_Robotech" package="2012-C" value="" x="20" y="15" rot="MR90"/>
+<element name="R2" library="Passive_Robotech" package="2012-R" value="10k" x="-2" y="11" rot="MR180"/>
+<element name="R3" library="Passive_Robotech" package="2012-R" value="10k" x="11" y="15" rot="MR90"/>
+<element name="R4" library="Passive_Robotech" package="2012-R" value="1k" x="10" y="9" rot="MR180"/>
+<element name="R5" library="Passive_Robotech" package="2012-R" value="1k" x="15" y="15" rot="MR180"/>
+<element name="C2" library="Passive_Robotech" package="2012-C" value="1n" x="14" y="11" rot="MR270"/>
+<element name="C11" library="Passive_Robotech" package="2012-C" value="1n" x="20" y="15" rot="MR90"/>
 <element name="IC2" library="IC_Robotech" package="MSOP8" value="7W14FU" x="23" y="12" rot="MR270"/>
 <element name="CON5" library="Connector_Robotech" package="5251-03-A" value="MOLEX-5251-03-A" x="26" y="3" rot="R180"/>
@@
 <element name="D2" library="Diode_Robotech" package="LED5" value="LED-5" x="77" y="10" rot="R270"/>
 <element name="R6" library="Passive_Robotech" package="2012-R" value="1kΩ" x="75" y="9" rot="MR270"/>
-<element name="R8" library="Passive_Robotech" package="2012-R" value="" x="10" y="5" rot="MR180"/>
-<element name="R9" library="Passive_Robotech" package="2012-R" value="" x="17" y="6" rot="MR180"/>
-<element name="C17" library="Passive_Robotech" package="2012-C" value="" x="21" y="5" rot="MR270"/>
+<element name="R8" library="Passive_Robotech" package="2012-R" value="10k" x="10" y="5" rot="MR180"/>
+<element name="R9" library="Passive_Robotech" package="2012-R" value="10k" x="17" y="6" rot="MR180"/>
+<element name="C17" library="Passive_Robotech" package="2012-C" value="0.1u" x="21" y="5" rot="MR270"/>
 <element name="CON7" library="Connector_Robotech" package="5251-02-S_LONG" value="MOLEX-5251-02-S_LONG" x="77" y="32" rot="R270"/>
 <element name="U$2" library="Document_Robotech" package="HOLE_3.2" value="" x="-7" y="3"/>
