File: Pawn.sch (EAGLE design)
At the start: 48 parts, among them CON2 MTDRV-A, CON26 MINI-USB-, CON27 UART-S, CON4 D-3500-4, CON5 MOLEX-5251-03-A, CON6 MOLEX-5251-03-A, CON7 MOLEX-5251-02-S_LONG, IC1 AZ1086H-3.3, IC2 7W14FU, IC8 R5F10JB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

Commit message: minor change
Parts:
- C11, C2: value (none) -> 1n
- C17: value (none) -> 0.1u
- R2, R3, R8, R9: value (none) -> 10k
- R4, R5: value (none) -> 1k
Other:
- note added: "ENC TIM2(CH1,CH2) MD TIM5(CH1)"
Changed lines of the file:
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@@
 <?xml version="1.0" encoding="utf-8"?>
 <!DOCTYPE eagle SYSTEM "eagle.dtd">
-<eagle version="8.5.1">
+<eagle version="8.3.1">
 <drawing>
 <settings>
@@
 <part name="CON4" library="Connector_Robotech" deviceset="D-3500-4" device=""/>
 <part name="P+9" library="Supply_Robotech" deviceset="+5V" device=""/>
-<part name="R2" library="Passive_Robotech" deviceset="R" device="-2012"/>
-<part name="R3" library="Passive_Robotech" deviceset="R" device="-2012"/>
-<part name="R4" library="Passive_Robotech" deviceset="R" device="-2012"/>
-<part name="R5" library="Passive_Robotech" deviceset="R" device="-2012"/>
-<part name="C2" library="Passive_Robotech" deviceset="C" device="-2012"/>
-<part name="C11" library="Passive_Robotech" deviceset="C" device="-2012"/>
+<part name="R2" library="Passive_Robotech" deviceset="R" device="-2012" value="10k"/>
+<part name="R3" library="Passive_Robotech" deviceset="R" device="-2012" value="10k"/>
+<part name="R4" library="Passive_Robotech" deviceset="R" device="-2012" value="1k"/>
+<part name="R5" library="Passive_Robotech" deviceset="R" device="-2012" value="1k"/>
+<part name="C2" library="Passive_Robotech" deviceset="C" device="-2012" value="1n"/>
+<part name="C11" library="Passive_Robotech" deviceset="C" device="-2012" value="1n"/>
 <part name="SUPPLY1" library="Supply_Robotech" deviceset="GND" device=""/>
 <part name="IC2" library="IC_Robotech" deviceset="7W14F" device="U"/>
@@
 <part name="SUPPLY15" library="Supply_Robotech" deviceset="GND" device=""/>
 <part name="P+13" library="Supply_Robotech" deviceset="+5V" device=""/>
-<part name="R8" library="Passive_Robotech" deviceset="R" device="-2012"/>
-<part name="R9" library="Passive_Robotech" deviceset="R" device="-2012"/>
-<part name="C17" library="Passive_Robotech" deviceset="C" device="-2012"/>
+<part name="R8" library="Passive_Robotech" deviceset="R" device="-2012" value="10k"/>
+<part name="R9" library="Passive_Robotech" deviceset="R" device="-2012" value="10k"/>
+<part name="C17" library="Passive_Robotech" deviceset="C" device="-2012" value="0.1u"/>
 <part name="SUPPLY16" library="Supply_Robotech" deviceset="GND" device=""/>
 <part name="P+14" library="Supply_Robotech" deviceset="+5V" device=""/>
@@
 <text x="469.9" y="-45.72" size="1.778" layer="91">NOかNCに注意！</text>
 <text x="492.76" y="127" size="1.778" layer="91">Arduino用USART2</text>
+<text x="236.22" y="106.68" size="1.778" layer="91">ENC TIM2(CH1,CH2)
+MD TIM5(CH1)</text>
 </plain>
 <instances>
